File: Advanced Linear Motor.kicad_pcb (KiCad board)
At the start: 6 copper layers, 200 x 95 mm, 10 parts, among them J1 Conn_01x03_Pin, J2 Conn_01x02_Pin

Commit message: 3 phase
Parts:
- moved J2 44.7 mm to (108.7, 80.0), turned to 90 degrees
- moved R1 9.20 mm to (93.1, 76.9)
- moved R2 9.20 mm to (93.1, 79.4)
- moved R3 9.20 mm to (93.1, 81.9)
- moved TH1 9.20 mm to (100.1, 78.9)
- moved J1 5.99 mm to (55.2, 85.6)
Routing:
- net Net-(J1-Pin_2): track 0.00 -> 7188.8 mm, vias 0 -> 10
- net Net-(J1-Pin_1): track 0.00 -> 7188.8 mm, vias 0 -> 10
- net Net-(J1-Pin_3): track 8719.7 -> 7188.8 mm, vias 12 -> 10

Commit message: v1_ready
Parts:
- moved H3 21.1 mm to (172.6, 58.2)
- moved H4 21.1 mm to (232.6, 58.2)
- moved H1 21.1 mm to (52.6, 58.2)
- moved H2 21.1 mm to (112.6, 58.2)
- moved R1 21.1 mm to (85.7, 57.1)
- moved R2 21.1 mm to (85.7, 59.6)
- moved R3 21.1 mm to (85.7, 62.1)
- moved TH1 21.1 mm to (92.7, 59.1)
- moved J1 21.1 mm to (47.8, 65.8)
- moved J2 21.1 mm to (101.3, 60.2)
Routing:
- net Net-(J1-Pin_3): track 7188.8 -> 14546.2 mm, vias 10 -> 20
- net Net-(J1-Pin_2): track 7188.8 -> 14546.2 mm, vias 10 -> 20
- net Net-(J1-Pin_1): track 7188.8 -> 14546.2 mm, vias 10 -> 20
